Commit message: update
1，修改由于命名空间导致的问题
2，更换爪子的controller为effort-controller
3，添加验证GPD是否安装正确的测试包
4，2022年04月22日15:07:13

File: package/dh_robotics_gripper/dh_robotics_ag95_gripper/dh_robotics_ag95_description/urdf/dh_robotics_ag95_gripper.urdf.xacro (robot description, xacro)
@@ -1,12 +1,13 @@
 <?xml version="1.0"?>
-<robot name="dh_robotics_ag95_gripper" xmlns:xacro="http://ros.org/wiki/xacro">
+<robot name="dh_robotics_ag95_gripper"
+    xmlns:xacro="http://ros.org/wiki/xacro">
     <xacro:include filename="$(find dh_robotics_ag95_description)/urdf/dh_robotics_ag95_gripper.transmission.xacro" />
     <xacro:macro name="dh_robotics_ag95_gripper" params="prefix parent *origin">
-        <joint name="${prefix}gripper_base_joint" type="fixed">
+        <joint name="gripper_base_joint" type="fixed">
             <parent link="${parent}"/>
-            <child link="${prefix}gripper_base_link"/>
+            <child link="gripper_base_link"/>
             <xacro:insert_block name="origin"/>
         </joint>
-        <link name="${prefix}gripper_base_link">
+        <link name="gripper_base_link">
             <visual>
                 <geometry>
@@ -27,27 +28,37 @@
             </inertial>
         </link>
-        <gazebo reference="${prefix}gripper_base_link">
-            <implicitSpringDamper>1</implicitSpringDamper>
-            <mu1>100000</mu1>
-            <mu2>100000</mu2>
-            <kp>100000000.0</kp>
-            <kd>1.0</kd>
-        </gazebo>
-        <joint name="${prefix}gripper_finger1_joint" type="revolute">
-            <parent link="${prefix}gripper_base_link"/>
-            <child link="${prefix}gripper_finger1_knuckle_link"/>
+        <gazebo reference="gripper_base_link">
+            <turnGravityOff>true</turnGravityOff>
+            <mu1>0.9</mu1>
+            <mu2>0.9</mu2>
+            <kp>100000000.0</kp>
+            <kd>1.0</kd>
+            <maxVel>0.0</maxVel>
+            <minDepth>0.001</minDepth>
+        </gazebo>
+        <joint name="gripper_finger1_joint" type="revolute">
+            <parent link="gripper_base_link"/>
+            <child link="gripper_finger1_knuckle_link"/>
             <axis xyz="0 -1 0"/>
             <origin rpy="0.0 0.0 ${pi}" xyz="-0.016 0 0.10586"/>
-            <limit lower="0.0" upper="0.65" velocity="2.0" effort="1000"/>
-        </joint>
-        <joint name="${prefix}gripper_finger2_joint" type="revolute">
-            <parent link="${prefix}gripper_base_link"/>
-            <child link="${prefix}gripper_finger2_knuckle_link"/>
+            <limit lower="0.0" upper="0.65" velocity="2.0" effort="1"/>
+            <dynamics damping="0.7"/>
+        </joint>
+        <gazebo reference="gripper_finger1_joint">
+            <implicitSpringDamper>1</implicitSpringDamper>
+        </gazebo>
+        <joint name="gripper_finger2_joint" type="revolute">
+            <parent link="gripper_base_link"/>
+            <child link="gripper_finger2_knuckle_link"/>
             <axis xyz="0 -1 0"/>
             <origin rpy="0.0 0.0 0.0" xyz="0.016  0 0.10586 "/>
-            <limit lower="-3.14" upper="3.14" velocity="100.0" effort="1000"/>
-            <mimic joint="${prefix}gripper_finger1_joint"/>
-        </joint>
-        <link name="${prefix}gripper_finger1_knuckle_link">
+            <limit lower="-3.14" upper="3.14" velocity="2.0" effort="1"/>
+            <mimic joint="gripper_finger1_joint"/>
+            <dynamics damping="0.7"/>
+        </joint>
+        <gazebo reference="gripper_finger2_joint">
+            <implicitSpringDamper>1</implicitSpringDamper>
+        </gazebo>
+        <link name="gripper_finger1_knuckle_link">
             <visual>
                 <geometry>
@@ -68,12 +79,14 @@
             </inertial>
         </link>
-        <gazebo reference="${prefix}gripper_finger1_knuckle_link">
-            <implicitSpringDamper>1</implicitSpringDamper>
-            <mu1>100000</mu1>
-            <mu2>100000</mu2>
-            <kp>100000000.0</kp>
-            <kd>1.0</kd>
-        </gazebo>
-        <link name="${prefix}gripper_finger2_knuckle_link">
+        <gazebo reference="gripper_finger1_knuckle_link">
+            <turnGravityOff>true</turnGravityOff>
+            <mu1>0.9</mu1>
+            <mu2>0.9</mu2>
+            <kp>100000000.0</kp>
+            <kd>1.0</kd>
+            <maxVel>0.0</maxVel>
+            <minDepth>0.001</minDepth>
+        </gazebo>
+        <link name="gripper_finger2_knuckle_link">
             <visual>
                 <geometry>
@@ -94,28 +107,38 @@
             </inertial>
         </link>
-        <gazebo reference="${prefix}gripper_finger2_knuckle_link">
-            <implicitSpringDamper>1</implicitSpringDamper>
-            <mu1>100000</mu1>
-            <mu2>100000</mu2>
-            <kp>100000000.0</kp>
-            <kd>1.0</kd>
-        </gazebo>
-        <joint name="${prefix}gripper_finger1_finger_joint" type="continuous">
-            <parent link="${prefix}gripper_finger1_knuckle_link"/>
-            <child link="${prefix}gripper_finger1_finger_link"/>
+        <gazebo reference="gripper_finger2_knuckle_link">
+            <turnGravityOff>true</turnGravityOff>
+            <mu1>0.9</mu1>
+            <mu2>0.9</mu2>
+            <kp>100000000.0</kp>
+            <kd>1.0</kd>
+            <maxVel>0.0</maxVel>
+            <minDepth>0.001</minDepth>
+        </gazebo>
+        <joint name="gripper_finger1_finger_joint" type="continuous">
+            <parent link="gripper_finger1_knuckle_link"/>
+            <child link="gripper_finger1_finger_link"/>
             <axis xyz="0 -1 0"/>
             <origin xyz="0.0292080077784 0.0 -0.0227132622407" rpy="0 0 0" />
-            <limit lower="-3.14" upper="3.14" velocity="100.0" effort="0.1"/>
-            <mimic joint="${prefix}gripper_finger1_joint" multiplier="0.4563942" offset="0"/>
-        </joint>
-        <joint name="${prefix}gripper_finger2_finger_joint" type="continuous">
-            <parent link="${prefix}gripper_finger2_knuckle_link"/>
-            <child link="${prefix}gripper_finger2_finger_link"/>
+            <limit lower="-3.14" upper="3.14" velocity="2.0" effort="1"/>
+            <mimic joint="gripper_finger1_joint" multiplier="0.4563942" offset="0"/>
+            <dynamics damping="0.7"/>
+        </joint>
+        <gazebo reference="gripper_finger1_finger_joint">
+            <implicitSpringDamper>1</implicitSpringDamper>
+        </gazebo>
+        <joint name="gripper_finger2_finger_joint" type="continuous">
+            <parent link="gripper_finger2_knuckle_link"/>
+            <child link="gripper_finger2_finger_link"/>
             <axis xyz="0 -1 0"/>
             <origin xyz="0.0292080077784 0.0 -0.0227132622407" rpy="0 0 0" />
-            <limit lower="-3.14" upper="3.14" velocity="100.0" effort="0.1"/>
-            <mimic joint="${prefix}gripper_finger1_joint" multiplier="0.4563942" offset="0"/>
-        </joint>
-        <link name="${prefix}gripper_finger1_finger_link">
+            <limit lower="-3.14" upper="3.14" velocity="2.0" effort="1"/>
+            <mimic joint="gripper_finger1_joint" multiplier="0.4563942" offset="0"/>
+            <dynamics damping="0.7"/>
+        </joint>
+        <gazebo reference="gripper_finger2_finger_joint">
+            <implicitSpringDamper>1</implicitSpringDamper>
+        </gazebo>
+        <link name="gripper_finger1_finger_link">
             <visual>
                 <geometry>
@@ -136,12 +159,14 @@
             </inertial>
         </link>
-        <gazebo reference="${prefix}gripper_finger1_finger_link">
-            <implicitSpringDamper>1</implicitSpringDamper>
-            <mu1>100000</mu1>
-            <mu2>100000</mu2>
-            <kp>100000000.0</kp>
-            <kd>1.0</kd>
-        </gazebo>
-        <link name="${prefix}gripper_finger2_finger_link">
+        <gazebo reference="gripper_finger1_finger_link">
+            <turnGravityOff>true</turnGravityOff>
+            <mu1>0.9</mu1>
+            <mu2>0.9</mu2>
+            <kp>100000000.0</kp>
+            <kd>1.0</kd>
+            <maxVel>0.0</maxVel>
+            <minDepth>0.001</minDepth>
+        </gazebo>
+        <link name="gripper_finger2_finger_link">
             <visual>
                 <geometry>
@@ -162,28 +187,38 @@
             </inertial>
         </link>
-        <gazebo reference="${prefix}gripper_finger2_finger_link">
-            <implicitSpringDamper>1</implicitSpringDamper>
-            <mu1>100000</mu1>
-            <mu2>100000</mu2>
-            <kp>100000000.0</kp>
-            <kd>1.0</kd>
-        </gazebo>
-        <joint name="${prefix}gripper_finger1_inner_knuckle_joint" type="continuous">
-            <parent link="${prefix}gripper_base_link"/>
-            <child link="${prefix}gripper_finger1_inner_knuckle_link"/>
+        <gazebo reference="gripper_finger2_finger_link">
+            <turnGravityOff>true</turnGravityOff>
+            <mu1>0.9</mu1>
+            <mu2>0.9</mu2>
+            <kp>100000000.0</kp>
+            <kd>1.0</kd>
+            <maxVel>0.0</maxVel>
+            <minDepth>0.001</minDepth>
+        </gazebo>
+        <joint name="gripper_finger1_inner_knuckle_joint" type="continuous">
+            <parent link="gripper_base_link"/>
+            <child link="gripper_finger1_inner_knuckle_link"/>
             <axis xyz="0 -1 0"/>
             <origin rpy="0.0 0.0 ${pi}" xyz="-0.016 0 0.10586"/>
-            <limit lower="-3.14" upper="3.14" velocity="100.0" effort="0.1"/>
-            <mimic joint="${prefix}gripper_finger1_joint" multiplier="1.49462955"  offset="0"/>
-        </joint>
-        <joint name="${prefix}gripper_finger2_inner_knuckle_joint" type="continuous">
-            <parent link="${prefix}gripper_base_link"/>
-            <child link="${prefix}gripper_finger2_inner_knuckle_link"/>
+            <limit lower="-3.14" upper="3.14" velocity="2.0" effort="1"/>
+            <mimic joint="gripper_finger1_joint" multiplier="1.49462955" offset="0"/>
+            <dynamics damping="0.7"/>
+        </joint>
+        <gazebo reference="gripper_finger1_inner_knuckle_joint">
+            <implicitSpringDamper>1</implicitSpringDamper>
+        </gazebo>
+        <joint name="gripper_finger2_inner_knuckle_joint" type="continuous">
+            <parent link="gripper_base_link"/>
+            <child link="gripper_finger2_inner_knuckle_link"/>
             <axis xyz="0 -1 0"/>
             <origin rpy="0.0 0.0 0.0" xyz="0.016 0 0.10586"/>
-            <limit lower="-3.14" upper="3.14" velocity="100.0" effort="0.1"/>
-            <mimic joint="${prefix}gripper_finger1_joint" multiplier="1.49462955" offset="0"/>
-        </joint>
-        <link name="${prefix}gripper_finger1_inner_knuckle_link">
+            <limit lower="-3.14" upper="3.14" velocity="2.0" effort="1"/>
+            <mimic joint="gripper_finger1_joint" multiplier="1.49462955" offset="0"/>
+            <dynamics damping="0.7"/>
+        </joint>
+        <gazebo reference="gripper_finger2_inner_knuckle_joint">
+            <implicitSpringDamper>1</implicitSpringDamper>
+        </gazebo>
+        <link name="gripper_finger1_inner_knuckle_link">
             <visual>
                 <geometry>
@@ -204,12 +239,14 @@
             </inertial>
         </link>
-        <gazebo reference="${prefix}gripper_finger1_inner_knuckle_link">
-            <implicitSpringDamper>1</implicitSpringDamper>
-            <mu1>100000</mu1>
-            <mu2>100000</mu2>
-            <kp>100000000.0</kp>
-            <kd>1.0</kd>
-        </gazebo>
-        <link name="${prefix}gripper_finger2_inner_knuckle_link">
+        <gazebo reference="gripper_finger1_inner_knuckle_link">
+            <turnGravityOff>true</turnGravityOff>
+            <mu1>0.9</mu1>
+            <mu2>0.9</mu2>
+            <kp>100000000.0</kp>
+            <kd>1.0</kd>
+            <maxVel>0.0</maxVel>
+            <minDepth>0.001</minDepth>
+        </gazebo>
+        <link name="gripper_finger2_inner_knuckle_link">
             <visual>
                 <geometry>
@@ -230,28 +267,38 @@
             </inertial>
         </link>
-        <gazebo reference="${prefix}gripper_finger2_inner_knuckle_link">
-            <implicitSpringDamper>1</implicitSpringDamper>
-            <mu1>100000</mu1>
-            <mu2>100000</mu2>
-            <kp>100000000.0</kp>
-            <kd>1.0</kd>
-        </gazebo>
-        <joint name="${prefix}gripper_finger1_finger_tip_joint" type="continuous">
-            <parent link="${prefix}gripper_finger1_inner_knuckle_link"/>
-            <child link="${prefix}gripper_finger1_finger_tip_link"/>
+        <gazebo reference="gripper_finger2_inner_knuckle_link">
+            <turnGravityOff>true</turnGravityOff>
+            <mu1>0.9</mu1>
+            <mu2>0.9</mu2>
+            <kp>100000000.0</kp>
+            <kd>1.0</kd>
+            <maxVel>0.0</maxVel>
+            <minDepth>0.001</minDepth>
+        </gazebo>
+        <joint name="gripper_finger1_finger_tip_joint" type="continuous">
+            <parent link="gripper_finger1_inner_knuckle_link"/>
+            <child link="gripper_finger1_finger_tip_link"/>
             <axis xyz="0 1 0"/>
             <origin xyz="0.0394969463769 0.0 0.0382752038125 " rpy="0.0 0.0 0.0"/>
-            <limit lower="-3.14" upper="3.14" velocity="100.0" effort="0.1"/>
-            <mimic joint="${prefix}gripper_finger1_joint" multiplier="1.49462955"/>
-        </joint>
-        <joint name="${prefix}gripper_finger2_finger_tip_joint" type="continuous">
-            <parent link="${prefix}gripper_finger2_inner_knuckle_link"/>
-            <child link="${prefix}gripper_finger2_finger_tip_link"/>
+            <limit lower="-3.14" upper="3.14" velocity="2.0" effort="1"/>
+            <mimic joint="gripper_finger1_joint" multiplier="1.49462955"/>
+            <dynamics damping="0.7"/>
+        </joint>
+        <gazebo reference="gripper_finger1_finger_tip_joint">
+            <implicitSpringDamper>1</implicitSpringDamper>
+        </gazebo>
+        <joint name="gripper_finger2_finger_tip_joint" type="continuous">
+            <parent link="gripper_finger2_inner_knuckle_link"/>
+            <child link="gripper_finger2_finger_tip_link"/>
             <axis xyz="0 1 0"/>
             <origin rpy="0.0 0.0 0.0" xyz="0.0394969463769  0.0 0.0382752038125  "/>
-            <limit lower="-3.14" upper="3.14" velocity="100.0" effort="0.1"/>
-            <mimic joint="${prefix}gripper_finger1_joint" multiplier="1.49462955"/>
-        </joint>
-        <link name="${prefix}gripper_finger1_finger_tip_link">
+            <limit lower="-3.14" upper="3.14" velocity="2.0" effort="1"/>
+            <mimic joint="gripper_finger1_joint" multiplier="1.49462955"/>
+            <dynamics damping="0.7"/>
+        </joint>
+        <gazebo reference="gripper_finger2_finger_tip_joint">
+            <implicitSpringDamper>1</implicitSpringDamper>
+        </gazebo>
+        <link name="gripper_finger1_finger_tip_link">
             <visual>
                 <geometry>
@@ -272,12 +319,14 @@
             </inertial>
         </link>
-        <gazebo reference="${prefix}gripper_finger1_finger_tip_link">
-            <implicitSpringDamper>1</implicitSpringDamper>
-            <mu1>100000</mu1>
-            <mu2>100000</mu2>
-            <kp>100000000.0</kp>
-            <kd>1.0</kd>
-        </gazebo>
-        <link name="${prefix}gripper_finger2_finger_tip_link">
+        <gazebo reference="gripper_finger1_finger_tip_link">
+            <turnGravityOff>true</turnGravityOff>
+            <mu1>0.9</mu1>
+            <mu2>0.9</mu2>
+            <kp>100000000.0</kp>
+            <kd>1.0</kd>
+            <maxVel>0.0</maxVel>
+            <minDepth>0.001</minDepth>
+        </gazebo>
+        <link name="gripper_finger2_finger_tip_link">
             <visual>
                 <geometry>
@@ -298,10 +347,12 @@
             </inertial>
         </link>
-        <gazebo reference="${prefix}gripper_finger2_finger_tip_link">
-            <implicitSpringDamper>1</implicitSpringDamper>
-            <mu1>100000</mu1>
-            <mu2>100000</mu2>
-            <kp>100000000.0</kp>
-            <kd>1.0</kd>
+        <gazebo reference="gripper_finger2_finger_tip_link">
+            <turnGravityOff>true</turnGravityOff>
+            <mu1>0.9</mu1>
+            <mu2>0.9</mu2>
+            <kp>100000000.0</kp>
+            <kd>1.0</kd>
+            <maxVel>0.0</maxVel>
+            <minDepth>0.001</minDepth>
         </gazebo>
         <gazebo>
@@ -310,18 +361,13 @@
                     <arm_name>gripper_arm</arm_name>
                     <palm_link>wrist_3_link</palm_link>
-                    <gripper_link>${prefix}gripper_finger1_finger_tip_link</gripper_link>
-                    <gripper_link>${prefix}gripper_finger2_finger_tip_link</gripper_link>
+                    <gripper_link>gripper_finger1_finger_tip_link</gripper_link>
+                    <gripper_link>gripper_finger2_finger_tip_link</gripper_link>
+                    <!-- <gripper_link>gripper_finger1_inner_knuckle_link</gripper_link> -->
+                    <!-- <gripper_link>gripper_finger2_inner_knuckle_link</gripper_link> -->
                 </arm>
-                <!-- <forces_angle_tolerance>100</forces_angle_tolerance>
-                <update_rate>4</update_rate>
-                <grip_count_threshold>4</grip_count_threshold>
-                <max_grip_count>8</max_grip_count>
-                <release_tolerance>0.005</release_tolerance>
-                <disable_collisions_on_attach>false</disable_collisions_on_attach>
-                <contact_topic>__default_topic__</contact_topic> -->
-                <forces_angle_tolerance>105</forces_angle_tolerance>
-                <update_rate>20</update_rate>
+                <forces_angle_tolerance>90</forces_angle_tolerance>
+                <update_rate>150</update_rate>
                 <grip_count_threshold>1</grip_count_threshold>
-                <max_grip_count>3</max_grip_count>
+                <max_grip_count>5</max_grip_count>
                 <release_tolerance>0.005</release_tolerance>
                 <disable_collisions_on_attach>true</disable_collisions_on_attach>
@@ -329,5 +375,5 @@
             </plugin>
         </gazebo>
-        <xacro:dh_robotics_ag95_gripper_transmission prefix="${prefix}" />
+        <xacro:dh_robotics_ag95_gripper_transmission prefix="" />
     </xacro:macro>
 </robot>

File: package/yixiuge_ur10_moveit_config/urdf/yixiuge_ur10.xacro (robot description, xacro)
@@ -6,5 +6,5 @@
   <!-- ur10 -->
   <xacro:include filename="$(find yixiuge_ur10_moveit_config)/urdf/yixiuge_ur10_description.xacro" />
-  <!-- arm -->
+  <!-- arm transmission -->
   <xacro:ur10_robot prefix="" joint_limited="false" transmission_hw_interface="$(arg transmission_hw_interface)"/>
   <!-- gripper -->
@@ -46,4 +46,8 @@
     </collision>
   </link>
+  <gazebo reference="camera_holder_link">
+    <selfCollide>true</selfCollide>
+    <turnGravityOff>true</turnGravityOff>
+  </gazebo>
   <joint name="camera_jiazi_joint" type="fixed">
     <origin xyz="0 0 0.004" rpy="0 0 0" />
@@ -72,4 +76,8 @@
     </inertial>
   </link>
+  <gazebo reference="camera_holder2_link">
+    <selfCollide>true</selfCollide>
+    <turnGravityOff>true</turnGravityOff>
+  </gazebo>
   <joint name="camera_jiazi_joint2" type="fixed">
     <origin xyz="0.0 -0.128 0.007" rpy="0 ${pi / 2} 0" />

File: package/yixiuge_ur10_moveit_config/urdf/yixiuge_ur10_description.xacro (robot description, xacro)
@@ -2,5 +2,5 @@
 <robot xmlns:xacro="http://wiki.ros.org/xacro">
   <xacro:include filename="$(find ur_description)/urdf/ur.transmission.xacro" />
-  <xacro:include filename="$(find ur_description)/urdf/ur.gazebo.xacro" />
+  <xacro:include filename="$(find yixiuge_ur10_moveit_config)/urdf/ur.gazebo.xacro" />
   <xacro:macro name="cylinder_inertial" params="radius length mass *origin">
     <inertial>
@@ -118,5 +118,5 @@
         </xacro:if>
       </xacro:if>
-      <dynamics damping="0.0" friction="0.0"/>
+      <dynamics damping="1.0" friction="1.0"/>
     </joint>
     <link name="${prefix}shoulder_link">
@@ -156,5 +156,5 @@
         </xacro:if>
       </xacro:if>
-      <dynamics damping="0.0" friction="0.0"/>
+      <dynamics damping="1.0" friction="1.0"/>
     </joint>
     <link name="${prefix}upper_arm_link">
@@ -194,5 +194,5 @@
         </xacro:if>
       </xacro:if>
-      <dynamics damping="0.0" friction="0.0"/>
+      <dynamics damping="1.0" friction="1.0"/>
     </joint>
     <link name="${prefix}forearm_link">
@@ -232,5 +232,5 @@
         </xacro:if>
       </xacro:if>
-      <dynamics damping="0.0" friction="0.0"/>
+      <dynamics damping="1.0" friction="1.0"/>
     </joint>
     <link name="${prefix}wrist_1_link">
@@ -270,5 +270,5 @@
         </xacro:if>
       </xacro:if>
-      <dynamics damping="0.0" friction="0.0"/>
+      <dynamics damping="1.0" friction="1.0"/>
     </joint>
     <link name="${prefix}wrist_2_link">
@@ -307,5 +307,5 @@
         </xacro:if>
       </xacro:if>
-      <dynamics damping="0.0" friction="0.0"/>
+      <dynamics damping="1.0" friction="1.0"/>
     </joint>
     <link name="${prefix}wrist_3_link">
